File: midi_sensor.sch (KiCad schematic (older format))
At the start: 45 parts, among them J1 Conn_01x12, Q1 BCX54, U1 CJ431, U2 LM393, U3 QRE1113, U4 LM321, U5 CJ431

Commit message: Add files via upload
Parts:
- removed J1: Conn_01x12, symbol Connector_Generic:Conn_01x12
- added J1: Conn_01x14, midi_sensor:edge_connector, symbol Connector_Generic:Conn_01x14
- C1, C2, C3, C4, C5, C6, C7: footprint (none) -> Capacitor_SMD:C_0603_1608Metric
- FID1, FID2: footprint (none) -> Fiducial:Fiducial_1mm_Mask2mm
- H1, H2: footprint (none) -> midi_sensor:hole_D3.5mm
- JP1, JP2, JP3, JP4, JP5, JP6: footprint (none) -> Jumper:SolderJumper-2_P1.3mm_Open_RoundedPad1.0x1.5mm
- R1, R10, R11, R12, R3, R4, R5, R6, R7, R8, R9: footprint (none) -> Resistor_SMD:R_0603_1608Metric
- R2: footprint (none) -> Resistor_SMD:R_2010_5025Metric
- TP1, TP2, TP3, TP4, TP5, TP6, TP7: footprint (none) -> midi_sensor:TP
- U2: footprint (none) -> Package_SO:SOIC-8_3.9x4.9mm_P1.27mm
Connections:
- net +5V: now also J1.11 (Pin_11), J1.12 (Pin_12)
- net +VCC_PULSE: now also J1.7 (Pin_7), J1.8 (Pin_8); no longer JP1.2 (B), JP2.2 (B), JP3.2 (B), JP4.2 (B), JP5.2 (B), JP6.2 (B)
- net COMP_OUT_HI: now also J1.14 (Pin_14)
- net COMP_OUT_LO: now also J1.13 (Pin_13)
- net GND: now also J1.10 (Pin_10), J1.9 (Pin_9)
- net GND_PULSE: now also JP1.2 (B), JP2.2 (B), JP3.2 (B), JP4.2 (B), JP5.2 (B), JP6.2 (B)
- net at JP1.1 (A): now also J1.1 (Pin_1)
- net at JP2.1 (A): now also J1.2 (Pin_2)
- net at JP3.1 (A): now also J1.3 (Pin_3)
- net at JP4.1 (A): now also J1.4 (Pin_4)
- net at JP5.1 (A): now also J1.5 (Pin_5)
- net at JP6.1 (A): now also J1.6 (Pin_6)
Other:
- moved on the sheet: C1, C3, JP1, JP2, JP3, JP4, JP5, JP6, TP2, U2C

Commit message: Add files via upload
Parts:
- removed D1, D2: BAT54C, Package_TO_SOT_SMD:SOT-23, symbol Diode:BAT54C
- removed Q1: BCX54, Package_TO_SOT_SMD:SOT-89-3, symbol Transistor_BJT:BCX56
- removed R12, R9: 13k, Resistor_SMD:R_0603_1608Metric, symbol Device:R
- added Q?: BC847, Package_TO_SOT_SMD:SOT-23, symbol Transistor_BJT:BC847
- R10: value 3.3k 1% -> 30k 1%
- R11: value 1.1 1% -> 13k 1%
- R2: value 4.7 1% 2010 -> 51 1%; footprint Resistor_SMD:R_2010_5025Metric -> (none)
- R4: value 1.1k -> 1k
- R7: value 1.1k 1% -> 30k 1%
- R8: value 1.1 1% -> 30k 1%
Connections:
- net COMP_OUT_HI: now also U2.1
- net COMP_OUT_LO: now also U2.7
- net at C2.1, R1.2, U1.2 (K): now also Q?.1 (B)
- net at U3.2 (K): now also Q?.3 (C)
- net at R2.1, TP4.1, U1.1 (REF): now also Q?.2 (E)
Changed lines of the file:
@@
 Sheet 1 1
 Title "Midi sensor"
-Date "2021-08-31"
-Rev "1.1"
+Date "2021-09-03"
+Rev "1.2"
 Comp "Yuriy Volkov"
 Comment1 ""
@@
 $EndComp
 $Comp
-L Transistor_BJT:BCX56 Q1
-U 1 1 612A1357
-P 3900 4200
-F 0 "Q1" H 4091 4246 50  0000 L CNN
-F 1 "BCX54" H 4091 4155 50  0000 L CNN
-F 2 "Package_TO_SOT_SMD:SOT-89-3" H 4100 4125 50  0001 L CIN
-F 3 "http://cache.nxp.com/documents/data_sheet/BCP56_BCX56_BC56PA.pdf?pspll=1" H 3900 4200 50  0001 L CNN
-	1    3900 4200
-	1    0    0    -1
-$EndComp
-$Comp
 L Amplifier_Operational:LM321 U4
 U 1 1 612A21D1
@@
 P 4000 4750
 F 0 "R2" H 4070 4796 50  0000 L CNN
-F 1 "4.7 1% 2010" H 4070 4705 50  0000 L CNN
-F 2 "Resistor_SMD:R_2010_5025Metric" V 3930 4750 50  0001 C CNN
+F 1 "51 1%" H 4070 4705 50  0000 L CNN
+F 2 "" V 3930 4750 50  0001 C CNN
 F 3 "~" H 4000 4750 50  0001 C CNN
 	1    4000 4750
@@
 P 6500 5250
 F 0 "R4" H 6570 5296 50  0000 L CNN
-F 1 "1.1k" H 6570 5205 50  0000 L CNN
+F 1 "1k" H 6570 5205 50  0000 L CNN
 F 2 "Resistor_SMD:R_0603_1608Metric" V 6430 5250 50  0001 C CNN
 F 3 "~" H 6500 5250 50  0001 C CNN
@@
 P 8000 2750
 F 0 "R7" H 8070 2796 50  0000 L CNN
-F 1 "1.1k 1%" H 8070 2705 50  0000 L CNN
+F 1 "30k 1%" H 8070 2705 50  0000 L CNN
 F 2 "Resistor_SMD:R_0603_1608Metric" V 7930 2750 50  0001 C CNN
 F 3 "~" H 8000 2750 50  0001 C CNN
@@
 P 8000 3350
 F 0 "R8" H 8070 3396 50  0000 L CNN
-F 1 "1.1 1%" H 8070 3305 50  0000 L CNN
+F 1 "30k 1%" H 8070 3305 50  0000 L CNN
 F 2 "Resistor_SMD:R_0603_1608Metric" V 7930 3350 50  0001 C CNN
 F 3 "~" H 8000 3350 50  0001 C CNN
@@
 P 9500 2750
 F 0 "R10" H 9570 2796 50  0000 L CNN
-F 1 "3.3k 1%" H 9570 2705 50  0000 L CNN
+F 1 "30k 1%" H 9570 2705 50  0000 L CNN
 F 2 "Resistor_SMD:R_0603_1608Metric" V 9430 2750 50  0001 C CNN
 F 3 "~" H 9500 2750 50  0001 C CNN
@@
 P 9500 3350
 F 0 "R11" H 9570 3396 50  0000 L CNN
-F 1 "1.1 1%" H 9570 3305 50  0000 L CNN
+F 1 "13k 1%" H 9570 3305 50  0000 L CNN
 F 2 "Resistor_SMD:R_0603_1608Metric" V 9430 3350 50  0001 C CNN
 F 3 "~" H 9500 3350 50  0001 C CNN
@@
 Wire Wire Line
 	8000 3000 8000 2900
-Wire Wire Line
-	8000 3200 8000 3100
 Connection ~ 8000 3000
 Wire Wire Line
@@
 Wire Wire Line
 	9500 3000 9500 2900
-Wire Wire Line
-	9500 3200 9500 3100
 Connection ~ 9500 3000
 Wire Wire Line
@@
 Text Label 9500 5000 2    50   ~ 0
 COMP_OUT_HI
-$Comp
-L Device:R R9
-U 1 1 6146A51C
-P 8800 3350
-F 0 "R9" H 8870 3396 50  0000 L CNN
-F 1 "13k" H 8870 3305 50  0000 L CNN
-F 2 "Resistor_SMD:R_0603_1608Metric" V 8730 3350 50  0001 C CNN
-F 3 "~" H 8800 3350 50  0001 C CNN
-	1    8800 3350
-	1    0    0    -1
-$EndComp
-$Comp
-L Device:R R12
-U 1 1 6146A964
-P 10300 3350
-F 0 "R12" H 10370 3396 50  0000 L CNN
-F 1 "13k" H 10370 3305 50  0000 L CNN
-F 2 "Resistor_SMD:R_0603_1608Metric" V 10230 3350 50  0001 C CNN
-F 3 "~" H 10300 3350 50  0001 C CNN
-	1    10300 3350
-	1    0    0    -1
-$EndComp
 Wire Wire Line
 	7500 2850 7500 3000
-Connection ~ 8000 3100
-Wire Wire Line
-	8000 3100 8000 3000
-Connection ~ 9500 3100
-Wire Wire Line
-	9500 3100 9500 3000
 $Comp
 L power:PWR_FLAG #FLG01
@@
 	0    1    -1   0
 $EndComp
-Wire Wire Line
-	9500 3100 10300 3100
-Wire Wire Line
-	8000 3100 8800 3100
-Wire Wire Line
-	10300 3500 10300 3800
-Wire Wire Line
-	8800 3500 8800 3800
 $Comp
 L Mechanical:Fiducial FID1
@@
 Wire Wire Line
 	5500 3200 5500 4000
-$Comp
-L Diode:BAT54C D1
-U 1 1 616FFA59
-P 8800 4100
-F 0 "D1" V 8754 4188 50  0000 L CNN
-F 1 "BAT54C" V 8845 4188 50  0000 L CNN
-F 2 "Package_TO_SOT_SMD:SOT-23" H 8875 4225 50  0001 L CNN
-F 3 "http://www.diodes.com/_files/datasheets/ds11005.pdf" H 8720 4100 50  0001 C CNN
-	1    8800 4100
-	0    1    1    0
-$EndComp
 Wire Wire Line
 	8000 4500 9500 4500
-$Comp
-L Diode:BAT54C D2
-U 1 1 6170CEAA
-P 10300 4100
-F 0 "D2" V 10254 4188 50  0000 L CNN
-F 1 "BAT54C" V 10345 4188 50  0000 L CNN
-F 2 "Package_TO_SOT_SMD:SOT-23" H 10375 4225 50  0001 L CNN
-F 3 "http://www.diodes.com/_files/datasheets/ds11005.pdf" H 10220 4100 50  0001 C CNN
-	1    10300 4100
-	0    1    1    0
-$EndComp
-Wire Wire Line
-	10300 5000 10300 4400
 Wire Wire Line
 	10300 5000 11000 5000
 Wire Wire Line
-	8800 5000 8800 4400
-Wire Wire Line
 	8800 5000 9500 5000
-Wire Wire Line
-	8800 3200 8800 3100
-Wire Wire Line
-	10300 3200 10300 3100
 Connection ~ 4000 6200
 Connection ~ 4000 5600
@@
 Wire Wire Line
 	1500 5600 2500 5600
+$Comp
+L Transistor_BJT:BC847 Q?
+U 1 1 613223B6
+P 3900 4200
+F 0 "Q?" H 4091 4246 50  0000 L CNN
+F 1 "BC847" H 4091 4155 50  0000 L CNN
+F 2 "Package_TO_SOT_SMD:SOT-23" H 4100 4125 50  0001 L CIN
+F 3 "http://www.infineon.com/dgdl/Infineon-BC847SERIES_BC848SERIES_BC849SERIES_BC850SERIES-DS-v01_01-en.pdf?fileId=db3a304314dca389011541d4630a1657" H 3900 4200 50  0001 L CNN
+	1    3900 4200
+	1    0    0    -1
+$EndComp
+Wire Wire Line
+	8000 3000 8000 3200
+Wire Wire Line
+	9500 3000 9500 3200
+Wire Wire Line
+	8600 4100 8800 4100
+Wire Wire Line
+	8800 4100 8800 5000
+Wire Wire Line
+	10100 4100 10300 4100
+Wire Wire Line
+	10300 4100 10300 5000
 $EndSCHEMATC

Commit message: Add files via upload
Parts:
- added G1: LOGO, midi_sensor:stamp, symbol stamp:LOGO
- H1, H2: footprint midi_sensor:hole_D3.5mm -> midi_sensor:hole_D2mm
- R2: footprint (none) -> Resistor_SMD:R_0603_1608Metric
- gave numbers to parts that had none: 1
- renumbered R11 to R10, R10 to R9
Changed lines of the file:
@@
 $EndDescr
 $Comp
-L stamp:LOGO #G1
+L stamp:LOGO G1
 U 1 1 6129F2D0
 P 10200 5950
-F 0 "#G1" H 10200 5828 60  0001 C CNN
+F 0 "G1" H 10200 5828 60  0001 C CNN
 F 1 "LOGO" H 10200 6072 60  0001 C CNN
-F 2 "" H 10200 5950 50  0001 C CNN
+F 2 "midi_sensor:stamp" H 10200 5950 50  0001 C CNN
 F 3 "" H 10200 5950 50  0001 C CNN
 	1    10200 5950
@@
 F 0 "H1" H 2100 7046 50  0000 L CNN
 F 1 "MountingHole" H 2100 6955 50  0000 L CNN
-F 2 "midi_sensor:hole_D3.5mm" H 2000 7000 50  0001 C CNN
+F 2 "midi_sensor:hole_D2mm" H 2000 7000 50  0001 C CNN
 F 3 "~" H 2000 7000 50  0001 C CNN
 	1    2000 7000
@@
 F 0 "R2" H 4070 4796 50  0000 L CNN
 F 1 "51 1%" H 4070 4705 50  0000 L CNN
-F 2 "" V 3930 4750 50  0001 C CNN
+F 2 "Resistor_SMD:R_0603_1608Metric" V 3930 4750 50  0001 C CNN
 F 3 "~" H 4000 4750 50  0001 C CNN
 	1    4000 4750
@@
 F 0 "H2" H 3100 7046 50  0000 L CNN
 F 1 "MountingHole" H 3100 6955 50  0000 L CNN
-F 2 "midi_sensor:hole_D3.5mm" H 3000 7000 50  0001 C CNN
+F 2 "midi_sensor:hole_D2mm" H 3000 7000 50  0001 C CNN
 F 3 "~" H 3000 7000 50  0001 C CNN
 	1    3000 7000
@@
 $EndComp
 $Comp
-L Device:R R10
+L Device:R R9
 U 1 1 613B758F
 P 9500 2750
-F 0 "R10" H 9570 2796 50  0000 L CNN
+F 0 "R9" H 9570 2796 50  0000 L CNN
 F 1 "30k 1%" H 9570 2705 50  0000 L CNN
 F 2 "Resistor_SMD:R_0603_1608Metric" V 9430 2750 50  0001 C CNN
@@
 $EndComp
 $Comp
-L Device:R R11
+L Device:R R10
 U 1 1 613B7803
 P 9500 3350
-F 0 "R11" H 9570 3396 50  0000 L CNN
+F 0 "R10" H 9570 3396 50  0000 L CNN
 F 1 "13k 1%" H 9570 3305 50  0000 L CNN
 F 2 "Resistor_SMD:R_0603_1608Metric" V 9430 3350 50  0001 C CNN
@@
 	1500 5600 2500 5600
 $Comp
-L Transistor_BJT:BC847 Q?
+L Transistor_BJT:BC847 Q1
 U 1 1 613223B6
 P 3900 4200
-F 0 "Q?" H 4091 4246 50  0000 L CNN
+F 0 "Q1" H 4091 4246 50  0000 L CNN
 F 1 "BC847" H 4091 4155 50  0000 L CNN
 F 2 "Package_TO_SOT_SMD:SOT-23" H 4100 4125 50  0001 L CIN
